File: Electrical/Driver Board/Tapper.brd (EAGLE design)
At the start: 71.9 x 31.4 mm, 30 parts, among them CN1 1X4-BIG, U10 DRV2605LDGS, U11 DRV2605LDGS, U12 TCA9548APWR, U3 DRV2605LDGS, U4 DRV2605LDGS, U5 DRV2605LDGS, U6 DRV2605LDGS, U7 DRV2605LDGS, U8 DRV2605LDGS, U9 DRV2605LDGS

Commit message: .
Parts:
- removed JP1: (no value), jumper:JP9Q
- added P1, P2, P3, P4, P5, P6, P7, P8, P9: B2B-PH-K, con-jst-ph:B2B-PH-K
- moved R5 21.6 mm to (15.0, 26.7), turned to 180 degrees
- moved C6 19.5 mm to (8.13, 22.4)
- moved C9 18.8 mm to (3.05, 10.7)
- moved U5 18.1 mm to (3.05, 6.86)
- moved RN1 16.3 mm to (30.2, 18.0), turned to 0 degrees
- moved JP2 16.0 mm to (57.4, 10.7), turned to 90 degrees
- moved U7 15.5 mm to (35.1, 7.11)
- moved C13 15.5 mm to (35.1, 10.9)
- moved C8 15.1 mm to (36.6, 17.8), turned to 270 degrees
- moved RN2 13.5 mm to (12.2, 17.0)
- moved U8 13.4 mm to (35.1, 24.4)
- moved C15 13.4 mm to (35.1, 28.2)
- moved C11 8.03 mm to (18.5, 10.7)
- moved U6 8.03 mm to (18.5, 6.86)
- moved C19 6.65 mm to (51.1, 20.1)
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Connections:
- net N$1: now also P2.2; no longer JP1.4
- net OUT+10: now also P6.1; no longer JP1.17
- net OUT+2: now also P1.1; no longer JP1.1
- net OUT+3: now also P2.1; no longer JP1.3
- net OUT+4: now also P3.1; no longer JP1.5
- net OUT+5: now also P4.1; no longer JP1.7
- net OUT+6: now also P5.1; no longer JP1.9
- net OUT+7: now also P9.1; no longer JP1.11
- net OUT+8: now also P8.1; no longer JP1.13
- net OUT+9: now also P7.1; no longer JP1.15
- net OUT-10: now also P6.2; no longer JP1.18
- net OUT-2: now also P1.2; no longer JP1.2
- net OUT-4: now also P3.2; no longer JP1.6
- net OUT-5: now also P4.2; no longer JP1.8
- net OUT-6: now also P5.2; no longer JP1.10
- net OUT-7: now also P9.2; no longer JP1.12
- net OUT-8: now also P8.2; no longer JP1.14
- net OUT-9: now also P7.2; no longer JP1.16
Other:
- board size 71.9 x 31.4 mm -> 69.6 x 28.6 mm
- board text added: "Tapper V0.3 (Dec 2021)"
- board text removed: "+"
- board text removed: "-"
- board text removed: "M0"
- board text removed: "M1"
- board text removed: "M2"
- board text removed: "M3"
- board text removed: "M4"
- board text removed: "M5"
- board text removed: "M6"
- board text removed: "M7"
- board text removed: "M8"
- board text removed: "Tapper V0.2 (Jun 2017)"

Commit message: .
Parts:
- turned P1 to 180 degrees
- turned P2 to 180 degrees
- turned P3 to 180 degrees
- turned P4 to 180 degrees
- turned P5 to 180 degrees
- turned P6 to 180 degrees
- turned P7 to 180 degrees
- turned P8 to 180 degrees
- turned P9 to 180 degrees
- turned U10 to 90 degrees
- turned U11 to 90 degrees
- turned U3 to 90 degrees
- turned U4 to 90 degrees
- turned U5 to 90 degrees
- turned U6 to 90 degrees
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
Commit message: .
Parts:
- moved R6 8.60 mm to (10.7, 26.7), turned to 0 degrees
- moved R10 5.73 mm to (20.6, 22.4), turned to 0 degrees
- moved C21 4.90 mm to (51.0, 6.28), turned to 0 degrees
- moved C13 4.70 mm to (35.1, 6.22), turned to 0 degrees
- moved C11 4.70 mm to (18.5, 5.97), turned to 0 degrees
- moved C19 4.70 mm to (51.1, 15.4), turned to 0 degrees
- moved C17 4.40 mm to (51.2, 24.0), turned to 0 degrees
- moved C15 4.00 mm to (35.0, 24.2), turned to 0 degrees
- moved C9 3.90 mm to (3.05, 6.77), turned to 0 degrees
- moved C7 3.90 mm to (3.05, 15.4), turned to 0 degrees
- moved C5 3.71 mm to (2.85, 24.5), turned to 0 degrees
- moved U3 3.70 mm to (2.95, 28.1)
- moved U4 3.30 mm to (3.05, 18.8)
- moved U5 3.30 mm to (3.05, 10.2)
- moved U8 3.20 mm to (35.0, 27.6)
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Connections:
- net +5V: now also U10.5, U11.5, U3.5, U4.5, U5.5, U6.5, U7.5, U8.5, U9.5
- net 2SCL: now also RN2.9; no longer RN2.7
- net 3SCL: now also RN2.7; no longer RN2.9
- net 4SCL: now also RN1.3; no longer RN1.2
- net 4SDA: now also RN1.4; no longer RN1.1
- net 5SCL: now also RN1.1; no longer RN1.4
- net 5SDA: now also RN1.2; no longer RN1.3
- net VIN: no longer RN1.5, RN2.10, U10.5, U11.5, U3.5, U4.5, U5.5, U6.5, U7.5, U8.5, U9.5
Routing:
- net +5V: track 0.00 -> 297.1 mm, vias 0 -> 6
- net GND: track 0.00 -> 255.6 mm, vias 0 -> 6
- net VIN: track 0.00 -> 105.1 mm, vias 0 -> 4
- net INPUTSCL: track 0.00 -> 88.3 mm, vias 0 -> 3
- net INPUTSDA: track 0.00 -> 85.5 mm
- net 3SDA: track 0.00 -> 35.7 mm, vias 0 -> 2
- net 3SCL: track 0.00 -> 33.3 mm, vias 0 -> 2
- net 1SCL: track 0.00 -> 23.6 mm
- net 1SDA: track 0.00 -> 23.4 mm
- net 2SDA: track 0.00 -> 18.3 mm
- net 0SCL: track 0.00 -> 15.5 mm
- net 0SDA: track 0.00 -> 14.9 mm
- net 2SCL: track 0.00 -> 14.0 mm
- net 6SDA: track 0.00 -> 10.7 mm
- net 4SDA: track 0.00 -> 9.18 mm
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
Commit message: 0.3v draft layout
Parts:
- RN1, RN2: value (none) -> 745C101332JP
- renumbered P1 to MI, P2 to M0, P3 to M1, P4 to M2, P5 to M3, P6 to M7, P7 to M6, P8 to M5, P9 to M4
Routing:
- net 7SCL: track 6.07 -> 43.6 mm
- net 5SCL: track 4.48 -> 40.9 mm, vias 0 -> 2
- net 7SDA: track 7.61 -> 43.8 mm
- net 5SDA: track 6.10 -> 41.0 mm, vias 0 -> 2
- net 6SCL: track 9.15 -> 33.3 mm, vias 0 -> 2
- net 6SDA: track 10.7 -> 32.4 mm, vias 0 -> 2
- net 4SDA: track 9.18 -> 24.8 mm, vias 0 -> 2
- net 4SCL: track 7.64 -> 22.4 mm, vias 0 -> 2
- net +5V: track 297.1 -> 310.3 mm, vias 6 -> 8
- net GND: track 255.6 -> 267.8 mm
- added copper zone on layer 16, net GND

Commit message: Board RC1
Parts:
- MI: value B2B-PH-K -> B2B-PH-K-S(LF)(SN)
- U12: value TCA9548APWR -> TCA9548APWR | PCA9548APW,118 | PI4MSD5V9547LEX
Routing:
- net 5SCL: track 40.9 -> 42.5 mm
Other:
- board text added: "3.3"
- board text added: "G"
- board text removed: "3.3V"
- board text removed: "5V"
- board text removed: "GND"
Changed lines of the file:
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@@
 <wire x1="60.432" y1="31.42" x2="-9.144" y2="31.42" width="0" layer="20"/>
 <wire x1="-9.144" y1="31.42" x2="-9.144" y2="2.794" width="0" layer="20"/>
-<text x="55.88" y="6.096" size="0.8128" layer="25" rot="R180">3.3V</text>
-<text x="54.61" y="7.874" size="0.8128" layer="25">5V</text>
-<text x="53.594" y="10.16" size="0.8128" layer="25">GND</text>
-<text x="55.118" y="12.7" size="0.8128" layer="25">D</text>
-<text x="55.118" y="15.494" size="0.8128" layer="25">C</text>
+<text x="58.68" y="5.396" size="0.8128" layer="25">3.3</text>
+<text x="58.794" y="10.36" size="0.8128" layer="25">G</text>
 <text x="58.928" y="27.94" size="0.8128" layer="25">C</text>
 <text x="58.928" y="25.4" size="0.8128" layer="25">D</text>
@@
 <text x="58.928" y="22.86" size="0.8128" layer="25">0</text>
 <text x="54.102" y="24.384" size="0.8128" layer="25" rot="R90">DISP</text>
-<text x="8.382" y="28.956" size="1.016" layer="25">Tapper V0.3 (Dec 2021)</text>
+<text x="6.882" y="30.056" size="1.016" layer="25">Tapper V0.3 (Dec 2021)</text>
+<text x="58.828" y="7.82" size="0.8128" layer="25">5</text>
+<text x="58.828" y="12.8" size="0.8128" layer="25">D</text>
+<text x="58.728" y="15.44" size="0.8128" layer="25">C</text>
 </plain>
 <attributes>
@@
 <attribute name="NAME" x="51.4" y="12.592" size="0.8128" layer="25" ratio="18" rot="R180"/>
 </element>
-<element name="U12" library="microbuilder" package="TSSOP24" value=" TCA9548APWR" x="20.828" y="16.764" smashed="yes" rot="R270">
+<element name="U12" library="microbuilder" package="TSSOP24" value=" TCA9548APWR | PCA9548APW,118 | PI4MSD5V9547LEX" x="20.828" y="16.764" smashed="yes" rot="R270">
 <attribute name="NAME" x="17.3992" y="20.8296" size="0.8128" layer="25" ratio="18"/>
 </element>
@@
 <element name="RN2" library="resistor-array" package="745-10NS" value="745C101332JP" x="12.192" y="17.018" smashed="yes" rot="R180">
 <attribute name="NAME" x="7.82" y="17.3785" size="1.016" layer="25" ratio="18" rot="R270"/>
-<attribute name="VALUE" x="7.747" y="19.2405" size="0.8128" layer="27" ratio="10" rot="R270"/>
 </element>
 <element name="RN1" library="resistor-array" package="745-10NS" value="745C101332JP" x="30.226" y="18.034" smashed="yes">
 <attribute name="NAME" x="33.4085" y="15.54" size="1.016" layer="25" ratio="18" rot="R180"/>
-<attribute name="VALUE" x="34.671" y="15.8115" size="0.8128" layer="27" ratio="10" rot="R90"/>
 </element>
 <element name="CN1" library="adafruit" library_urn="urn:adsk.eagle:library:420" package="1X04-BIG" value="1X4-BIG" x="57.404" y="20.828" smashed="yes" rot="R90"/>
-<element name="MI" library="con-jst-ph" package="B2B-PH-K" value="B2B-PH-K" x="-4.318" y="26.416" smashed="yes" rot="R180">
+<element name="MI" library="con-jst-ph" package="B2B-PH-K" value="B2B-PH-K-S(LF)(SN)" x="-4.318" y="26.416" smashed="yes" rot="R180">
 <attribute name="LABEL" value="" x="-4.318" y="26.416" size="1.778" layer="27" rot="R180" display="off"/>
 <attribute name="NAME" x="-1.397" y="24.13" size="1.016" layer="25" ratio="18" rot="R180"/>
@@
 <wire x1="53.772" y1="14.3" x2="57.404" y2="10.668" width="0.2032" layer="1"/>
 <wire x1="51.17" y1="14.3" x2="53.3" y2="14.3" width="0.2032" layer="1"/>
+<wire x1="53.772" y1="14.3" x2="53.8" y2="14.3" width="0.2032" layer="1"/>
 <wire x1="53.3" y1="14.3" x2="53.772" y2="14.3" width="0.2032" layer="1"/>
-<wire x1="53.254" y1="15.446" x2="53.3" y2="15.4" width="0.2032" layer="1"/>
 <wire x1="54.0842125" y1="18.896" x2="54.233" y2="18.7472125" width="0.2032" layer="1"/>
-<wire x1="53.254" y1="16.1131" x2="53.254" y2="15.446" width="0.2032" layer="1"/>
+<wire x1="53.8" y1="16.6591" x2="53.8" y2="14.3" width="0.2032" layer="1"/>
 <wire x1="53.254" y1="19.002" x2="53.36" y2="18.896" width="0.2032" layer="1"/>
 <wire x1="53.36" y1="18.896" x2="54.0842125" y2="18.896" width="0.2032" layer="1"/>
 <wire x1="54.233" y1="18.7472125" x2="54.233" y2="17.0921" width="0.2032" layer="1"/>
-<wire x1="54.233" y1="17.0921" x2="53.254" y2="16.1131" width="0.2032" layer="1"/>
-<wire x1="53.3" y1="15.4" x2="53.3" y2="14.3" width="0.2032" layer="1"/>
+<wire x1="54.233" y1="17.0921" x2="53.8" y2="16.6591" width="0.2032" layer="1"/>
 <wire x1="53.7692125" y1="23.9" x2="54.5" y2="23.9" width="0.2032" layer="1"/>
 <wire x1="52.9132125" y1="23.044" x2="53.7692125" y2="23.9" width="0.2032" layer="1"/>
@@
 <wire x1="37.1089" y1="25.44395" x2="45.14165" y2="25.44395" width="0.127" layer="16"/>
 <wire x1="31.9913" y1="20.32635" x2="37.1089" y2="25.44395" width="0.127" layer="16"/>
-<wire x1="31.9913" y1="17.39265" x2="31.9913" y2="20.32635" width="0.127" layer="16"/>
-<wire x1="28.5973" y1="13.99865" x2="31.9913" y2="17.39265" width="0.127" layer="16"/>
-<wire x1="27.03045" y1="13.99865" x2="28.5973" y2="13.99865" width="0.127" layer="16"/>
-<wire x1="25.73195" y1="15.29715" x2="27.03045" y2="13.99865" width="0.127" layer="16"/>
+<wire x1="31.9913" y1="16.59265" x2="31.9913" y2="20.32635" width="0.127" layer="16"/>
+<wire x1="28.8973" y1="13.49865" x2="31.9913" y2="16.59265" width="0.127" layer="16"/>
+<wire x1="26.43045" y1="13.49865" x2="28.8973" y2="13.49865" width="0.127" layer="16"/>
+<wire x1="26.43045" y1="13.49865" x2="25.73195" y2="14.19715" width="0.127" layer="16"/>
+<wire x1="25.73195" y1="15.29715" x2="25.73195" y2="14.19715" width="0.127" layer="16"/>
 <wire x1="25.73195" y1="16.4465" x2="25.73195" y2="15.29715" width="0.127" layer="1"/>
 <wire x1="53.3654" y1="26.9621" x2="53.408" y2="26.992" width="0.127" layer="1"/>

Commit message: More improvements
Parts:
- removed CN1: 1X4-BIG, adafruit:1X04-BIG
- removed JP2: (no value), microbuilder:1X05_ROUND_FULL_76
- added P1: B5B-PH-K, con-jst-ph:B5B-PH-K
- added P2: B4B-PH-K, con-jst-ph:B4B-PH-K
Connections:
- net +5V: now also P1.2, P2.1; no longer CN1.1, JP2.2
- net GND: now also P1.3, P2.2; no longer CN1.2, JP2.3
- net INPUTSCL: now also P1.5, P2.4; no longer CN1.4, JP2.5
- net INPUTSDA: now also P1.4, P2.3; no longer CN1.3, JP2.4
- net VIN: now also P1.1; no longer JP2.1
Routing:
- net GND: track 267.5 -> 241.0 mm
- net +5V: track 310.3 -> 302.3 mm
- net INPUTSDA: track 85.5 -> 87.3 mm
- net 3SDA: track 35.7 -> 37.1 mm
- net INPUTSCL: track 88.3 -> 89.1 mm
- net VIN: track 105.1 -> 105.8 mm
- net 3SCL: track 33.3 -> 33.9 mm
Other:
- board text added: "uC"

Commit message: v0.31: Minor routing tweak
Routing:
- net GND: track 241.0 -> 216.1 mm
Other:
- board text added: "Tapper V0.31 (Jan 2021)"
- board text removed: "Tapper V0.3 (Dec 2021)"
Changed lines of the file:
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@@
 <text x="54.228" y="23.46" size="0.8128" layer="25">0</text>
 <text x="55.102" y="30.284" size="0.8128" layer="25">DISP</text>
-<text x="6.882" y="30.056" size="1.016" layer="25">Tapper V0.3 (Dec 2021)</text>
+<text x="6.882" y="30.056" size="1.016" layer="25">Tapper V0.31 (Jan 2021)</text>
 <text x="54.228" y="7.82" size="0.8128" layer="25">5</text>
 <text x="54.128" y="11.8" size="0.8128" layer="25">D</text>
@@
 <wire x1="2.098" y1="9.6322125" x2="2.098" y2="6.768" width="0.2032" layer="1"/>
 <wire x1="23.7458" y1="18.389" x2="23.0081" y2="18.389" width="0.2032" layer="1"/>
-<wire x1="21.6971" y1="19.7" x2="20.2" y2="19.7" width="0.2032" layer="1"/>
-<via x="20.2" y="19.7" extent="1-16" drill="0.35"/>
-<wire x1="20.2" y1="19.7" x2="17.2" y2="19.7" width="0.2032" layer="16"/>
-<wire x1="17.2" y1="19.7" x2="16.65" y2="20.25" width="0.2032" layer="16"/>
+<wire x1="22.9971" y1="18.4" x2="21.7" y2="18.4" width="0.2032" layer="1"/>
+<via x="21.7" y="18.4" extent="1-16" drill="0.35"/>
 <via x="16.2" y="20.3" extent="1-16" drill="0.35"/>
-<wire x1="16.45" y1="20.05" x2="16.2" y2="20.3" width="0.2032" layer="16"/>
 <wire x1="16.2" y1="20.3" x2="16.239" y2="20.339" width="0.2032" layer="1"/>
 <wire x1="16.239" y1="20.339" x2="17.9102" y2="20.339" width="0.2032" layer="1"/>
-<wire x1="23.0081" y1="18.389" x2="21.6971" y2="19.7" width="0.2032" layer="1"/>
+<wire x1="23.0081" y1="18.389" x2="22.9971" y2="18.4" width="0.2032" layer="1"/>
 <wire x1="17.592" y1="5.968" x2="16.824" y2="5.2" width="0.2032" layer="1"/>
 <wire x1="16.824" y1="5.2" x2="10.8" y2="5.2" width="0.2032" layer="1"/>
@@
 <via x="53.7" y="23.9" extent="1-16" drill="0.35"/>
 <wire x1="34.002" y1="24.194" x2="32.506" y2="24.194" width="0.2032" layer="1"/>
-<wire x1="32.506" y1="24.194" x2="32.2" y2="24.5" width="0.2032" layer="1"/>
-<wire x1="32.2" y1="24.5" x2="29.4558125" y2="24.5" width="0.2032" layer="1"/>
-<wire x1="29.4558125" y1="24.5" x2="29.4462125" y2="24.4904" width="0.2032" layer="1"/>
-<wire x1="23.7" y1="24.7" x2="23.9096" y2="24.4904" width="0.2032" layer="1"/>
-<wire x1="29.4462125" y1="24.4904" x2="23.9096" y2="24.4904" width="0.2032" layer="1"/>
-<via x="23.7" y="24.7" extent="1-16" drill="0.35"/>
-<wire x1="18.16186875" y1="24.7322" x2="17.63813125" y2="24.7322" width="0.2032" layer="16"/>
-<wire x1="17.63813125" y1="24.7322" x2="17.2678" y2="24.36186875" width="0.2032" layer="16"/>
-<wire x1="18.19406875" y1="24.7" x2="18.16186875" y2="24.7322" width="0.2032" layer="16"/>
-<wire x1="17.2678" y1="20.8678" x2="16.65" y2="20.25" width="0.2032" layer="16"/>
-<wire x1="16.65" y1="20.25" x2="16.45" y2="20.05" width="0.2032" layer="16"/>
-<wire x1="17.2678" y1="24.36186875" x2="17.2678" y2="20.8678" width="0.2032" layer="16"/>
-<wire x1="23.7" y1="24.7" x2="18.19406875" y2="24.7" width="0.2032" layer="16"/>
+<wire x1="31.6" y1="25.4" x2="31.6" y2="25.1" width="0.2032" layer="1"/>
+<wire x1="32.506" y1="24.194" x2="31.6" y2="25.1" width="0.2032" layer="1"/>
+<via x="31.6" y="25.4" extent="1-16" drill="0.35"/>
 <wire x1="2.2352" y1="10.68705" x2="5.23875" y2="10.68705" width="0.2032" layer="1"/>
 <wire x1="5.23875" y1="10.68705" x2="5.248" y2="10.658" width="0.2032" layer="1"/>

Commit message: i2c bus chip PI4MSD5V9547LEX is NOT the same as TCA9548APWR. It may be made to run similar, but, for instance, it has a different control register that doesnt allow for simultaneous writing to multiple busses
Parts:
- U12: value TCA9548APWR | PCA9548APW,118 | PI4MSD5V9547LEX -> TCA9548APWR | PCA9548APW,118
Changed lines of the file:
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@@
 <attribute name="NAME" x="51.4" y="12.592" size="0.8128" layer="25" ratio="18" rot="R180"/>
 </element>
-<element name="U12" library="microbuilder" package="TSSOP24" value=" TCA9548APWR | PCA9548APW,118 | PI4MSD5V9547LEX" x="20.828" y="16.764" smashed="yes" rot="R270">
+<element name="U12" library="microbuilder" package="TSSOP24" value=" TCA9548APWR | PCA9548APW,118" x="20.828" y="16.764" smashed="yes" rot="R270">
 <attribute name="NAME" x="17.3992" y="20.8296" size="0.8128" layer="25" ratio="18"/>
 </element>
