File: Electrical/Driver Board/Tapper.sch (EAGLE design)
At the start: 30 parts, among them CN1 1X4-BIG, U10 DRV2605LDGS, U11 DRV2605LDGS, U12 TCA9548APWR, U3 DRV2605LDGS, U4 DRV2605LDGS, U5 DRV2605LDGS, U6 DRV2605LDGS, U7 DRV2605LDGS, U8 DRV2605LDGS, U9 DRV2605LDGS

Commit message: .
Parts:
- removed JP1: (no value), jumper:JP9QE
- added P1, P2, P3, P4, P5, P6, P7, P8, P9: B2B-PH-K, con-jst-ph:B2B-PH-K
Connections:
- net N$1: now also P2.2; no longer JP1-2.2
- net OUT+10: now also P6.1; no longer JP1-9.1
- net OUT+2: now also P1.1; no longer JP1-1.1
- net OUT+3: now also P2.1; no longer JP1-2.1
- net OUT+4: now also P3.1; no longer JP1-3.1
- net OUT+5: now also P4.1; no longer JP1-4.1
- net OUT+6: now also P5.1; no longer JP1-5.1
- net OUT+7: now also P9.1; no longer JP1-6.1
- net OUT+8: now also P8.1; no longer JP1-7.1
- net OUT+9: now also P7.1; no longer JP1-8.1
- net OUT-10: now also P6.2; no longer JP1-9.2
- net OUT-2: now also P1.2; no longer JP1-1.2
- net OUT-4: now also P3.2; no longer JP1-3.2
- net OUT-5: now also P4.2; no longer JP1-4.2
- net OUT-6: now also P5.2; no longer JP1-5.2
- net OUT-7: now also P9.2; no longer JP1-6.2
- net OUT-8: now also P8.2; no longer JP1-7.2
- net OUT-9: now also P7.2; no longer JP1-8.2

Commit message: .
Connections:
- net +5V: now also U10.EN, U11.EN, U3.EN, U4.EN, U5.EN, U6.EN, U7.EN, U8.EN, U9.EN
- net 2SCL: now also RN2.9; no longer RN2.7
- net 3SCL: now also RN2.7; no longer RN2.9
- net 4SCL: now also RN1.3; no longer RN1.2
- net 4SDA: now also RN1.4; no longer RN1.1
- net 5SCL: now also RN1.1; no longer RN1.4
- net 5SDA: now also RN1.2; no longer RN1.3
- net VIN: no longer RN1.5, RN2.10, U10.EN, U11.EN, U3.EN, U4.EN, U5.EN, U6.EN, U7.EN, U8.EN, U9.EN

Commit message: 0.3v draft layout
Parts:
- RN1, RN2: value (none) -> 745C101332JP
- renumbered P1 to MI, P2 to M0, P3 to M1, P4 to M2, P5 to M3, P6 to M7, P7 to M6, P8 to M5, P9 to M4
Changed lines of the file:
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@@
 <part name="U$6" library="microbuilder" deviceset="GND" device=""/>
 <part name="U$7" library="microbuilder" deviceset="GND" device=""/>
-<part name="RN2" library="resistor-array" deviceset="745-10" device="NS"/>
+<part name="RN2" library="resistor-array" deviceset="745-10" device="NS" value="745C101332JP"/>
 <part name="U$9" library="microbuilder" deviceset="VIN" device=""/>
-<part name="RN1" library="resistor-array" deviceset="745-10" device="NS"/>
+<part name="RN1" library="resistor-array" deviceset="745-10" device="NS" value="745C101332JP"/>
 <part name="U$3" library="microbuilder" deviceset="VIN" device=""/>
 <part name="P+1" library="supply1" library_urn="urn:adsk.eagle:library:371" deviceset="+5V" device=""/>
@@
 <part name="U$17" library="microbuilder" deviceset="GND" device=""/>
 <part name="U$18" library="microbuilder" deviceset="GND" device=""/>
-<part name="P1" library="con-jst-ph" deviceset="B2B-PH-K" device=""/>
-<part name="P2" library="con-jst-ph" deviceset="B2B-PH-K" device=""/>
-<part name="P3" library="con-jst-ph" deviceset="B2B-PH-K" device=""/>
-<part name="P4" library="con-jst-ph" deviceset="B2B-PH-K" device=""/>
-<part name="P5" library="con-jst-ph" deviceset="B2B-PH-K" device=""/>
-<part name="P6" library="con-jst-ph" deviceset="B2B-PH-K" device=""/>
-<part name="P7" library="con-jst-ph" deviceset="B2B-PH-K" device=""/>
-<part name="P8" library="con-jst-ph" deviceset="B2B-PH-K" device=""/>
-<part name="P9" library="con-jst-ph" deviceset="B2B-PH-K" device=""/>
+<part name="MI" library="con-jst-ph" deviceset="B2B-PH-K" device=""/>
+<part name="M0" library="con-jst-ph" deviceset="B2B-PH-K" device=""/>
+<part name="M1" library="con-jst-ph" deviceset="B2B-PH-K" device=""/>
+<part name="M2" library="con-jst-ph" deviceset="B2B-PH-K" device=""/>
+<part name="M3" library="con-jst-ph" deviceset="B2B-PH-K" device=""/>
+<part name="M7" library="con-jst-ph" deviceset="B2B-PH-K" device=""/>
+<part name="M6" library="con-jst-ph" deviceset="B2B-PH-K" device=""/>
+<part name="M5" library="con-jst-ph" deviceset="B2B-PH-K" device=""/>
+<part name="M4" library="con-jst-ph" deviceset="B2B-PH-K" device=""/>
 <part name="P+12" library="supply1" library_urn="urn:adsk.eagle:library:371" deviceset="+5V" device=""/>
 <part name="P+13" library="supply1" library_urn="urn:adsk.eagle:library:371" deviceset="+5V" device=""/>
@@
 <attribute name="VALUE" x="199.136" y="96.52" size="1.27" layer="96"/>
 </instance>
-<instance part="P1" gate="G$1" x="144.78" y="139.7" smashed="yes">
+<instance part="MI" gate="G$1" x="144.78" y="139.7" smashed="yes">
 <attribute name="NAME" x="143.51" y="142.875" size="1.778" layer="95"/>
 <attribute name="VALUE" x="143.51" y="132.08" size="1.778" layer="95"/>
 </instance>
-<instance part="P2" gate="G$1" x="144.78" y="93.98" smashed="yes">
+<instance part="M0" gate="G$1" x="144.78" y="93.98" smashed="yes">
 <attribute name="NAME" x="143.51" y="97.155" size="1.778" layer="95"/>
 <attribute name="VALUE" x="143.51" y="86.36" size="1.778" layer="95"/>
 </instance>
-<instance part="P3" gate="G$1" x="147.32" y="50.8" smashed="yes">
+<instance part="M1" gate="G$1" x="147.32" y="50.8" smashed="yes">
 <attribute name="NAME" x="146.05" y="53.975" size="1.778" layer="95"/>
 <attribute name="VALUE" x="146.05" y="43.18" size="1.778" layer="95"/>
 </instance>
-<instance part="P4" gate="G$1" x="147.32" y="10.16" smashed="yes">
+<instance part="M2" gate="G$1" x="147.32" y="10.16" smashed="yes">
 <attribute name="NAME" x="146.05" y="13.335" size="1.778" layer="95"/>
 <attribute name="VALUE" x="146.05" y="2.54" size="1.778" layer="95"/>
 </instance>
-<instance part="P5" gate="G$1" x="147.32" y="-30.48" smashed="yes">
+<instance part="M3" gate="G$1" x="147.32" y="-30.48" smashed="yes">
 <attribute name="NAME" x="146.05" y="-27.305" size="1.778" layer="95"/>
 <attribute name="VALUE" x="146.05" y="-38.1" size="1.778" layer="95"/>
 </instance>
-<instance part="P6" gate="G$1" x="241.3" y="-15.24" smashed="yes">
+<instance part="M7" gate="G$1" x="241.3" y="-15.24" smashed="yes">
 <attribute name="NAME" x="240.03" y="-12.065" size="1.778" layer="95"/>
 <attribute name="VALUE" x="240.03" y="-22.86" size="1.778" layer="95"/>
 </instance>
-<instance part="P7" gate="G$1" x="241.3" y="27.94" smashed="yes">
+<instance part="M6" gate="G$1" x="241.3" y="27.94" smashed="yes">
 <attribute name="NAME" x="240.03" y="31.115" size="1.778" layer="95"/>
 <attribute name="VALUE" x="240.03" y="20.32" size="1.778" layer="95"/>
 </instance>
-<instance part="P8" gate="G$1" x="241.3" y="68.58" smashed="yes">
+<instance part="M5" gate="G$1" x="241.3" y="68.58" smashed="yes">
 <attribute name="NAME" x="240.03" y="71.755" size="1.778" layer="95"/>
 <attribute name="VALUE" x="240.03" y="60.96" size="1.778" layer="95"/>
 </instance>
-<instance part="P9" gate="G$1" x="241.3" y="111.76" smashed="yes">
+<instance part="M4" gate="G$1" x="241.3" y="111.76" smashed="yes">
 <attribute name="NAME" x="240.03" y="114.935" size="1.778" layer="95"/>
 <attribute name="VALUE" x="240.03" y="104.14" size="1.778" layer="95"/>
@@
 <pinref part="U3" gate="G$1" pin="OUT+"/>
 <wire x1="132.08" y1="139.7" x2="139.7" y2="139.7" width="0.1524" layer="91"/>
-<pinref part="P1" gate="G$1" pin="1"/>
+<pinref part="MI" gate="G$1" pin="1"/>
 </segment>
 </net>
@@
 <pinref part="U3" gate="G$1" pin="OUT-"/>
 <wire x1="132.08" y1="137.16" x2="139.7" y2="137.16" width="0.1524" layer="91"/>
-<pinref part="P1" gate="G$1" pin="2"/>
+<pinref part="MI" gate="G$1" pin="2"/>
 </segment>
 </net>
@@
 <pinref part="U4" gate="G$1" pin="OUT+"/>
 <wire x1="132.08" y1="93.98" x2="139.7" y2="93.98" width="0.1524" layer="91"/>
-<pinref part="P2" gate="G$1" pin="1"/>
+<pinref part="M0" gate="G$1" pin="1"/>
 <wire x1="139.7" y1="93.98" x2="140.462" y2="93.98" width="0.1524" layer="91"/>
 <junction x="139.7" y="93.98"/>
@@
 <pinref part="U5" gate="G$1" pin="OUT+"/>
 <wire x1="132.08" y1="50.8" x2="142.24" y2="50.8" width="0.1524" layer="91"/>
-<pinref part="P3" gate="G$1" pin="1"/>
+<pinref part="M1" gate="G$1" pin="1"/>
 </segment>
 </net>
@@
 <pinref part="U5" gate="G$1" pin="OUT-"/>
 <wire x1="132.08" y1="48.26" x2="142.24" y2="48.26" width="0.1524" layer="91"/>
-<pinref part="P3" gate="G$1" pin="2"/>
+<pinref part="M1" gate="G$1" pin="2"/>
 </segment>
 </net>
@@
 <pinref part="U6" gate="G$1" pin="OUT+"/>
 <wire x1="132.08" y1="10.16" x2="142.24" y2="10.16" width="0.1524" layer="91"/>
-<pinref part="P4" gate="G$1" pin="1"/>
+<pinref part="M2" gate="G$1" pin="1"/>
 </segment>
 </net>
@@
 <pinref part="U6" gate="G$1" pin="OUT-"/>
 <wire x1="132.08" y1="7.62" x2="142.24" y2="7.62" width="0.1524" layer="91"/>
-<pinref part="P4" gate="G$1" pin="2"/>
+<pinref part="M2" gate="G$1" pin="2"/>
 </segment>
 </net>
@@
 <pinref part="U7" gate="G$1" pin="OUT+"/>
 <wire x1="132.08" y1="-30.48" x2="142.24" y2="-30.48" width="0.1524" layer="91"/>
-<pinref part="P5" gate="G$1" pin="1"/>
+<pinref part="M3" gate="G$1" pin="1"/>
 </segment>
 </net>
@@
 <pinref part="U7" gate="G$1" pin="OUT-"/>
 <wire x1="132.08" y1="-33.02" x2="142.24" y2="-33.02" width="0.1524" layer="91"/>
-<pinref part="P5" gate="G$1" pin="2"/>
+<pinref part="M3" gate="G$1" pin="2"/>
 </segment>
 </net>
@@
 <pinref part="U8" gate="G$1" pin="OUT+"/>
 <wire x1="226.06" y1="111.76" x2="236.22" y2="111.76" width="0.1524" layer="91"/>
-<pinref part="P9" gate="G$1" pin="1"/>
+<pinref part="M4" gate="G$1" pin="1"/>
 </segment>
 </net>
@@
 <pinref part="U8" gate="G$1" pin="OUT-"/>
 <wire x1="226.06" y1="109.22" x2="236.22" y2="109.22" width="0.1524" layer="91"/>
-<pinref part="P9" gate="G$1" pin="2"/>
+<pinref part="M4" gate="G$1" pin="2"/>
 </segment>
 </net>
@@
 <pinref part="U9" gate="G$1" pin="OUT+"/>
 <wire x1="226.06" y1="68.58" x2="236.22" y2="68.58" width="0.1524" layer="91"/>
-<pinref part="P8" gate="G$1" pin="1"/>
+<pinref part="M5" gate="G$1" pin="1"/>
 </segment>
 </net>
@@
 <pinref part="U9" gate="G$1" pin="OUT-"/>
 <wire x1="226.06" y1="66.04" x2="236.22" y2="66.04" width="0.1524" layer="91"/>
-<pinref part="P8" gate="G$1" pin="2"/>
+<pinref part="M5" gate="G$1" pin="2"/>
 </segment>
 </net>
@@
 <pinref part="U10" gate="G$1" pin="OUT+"/>
 <wire x1="226.06" y1="27.94" x2="236.22" y2="27.94" width="0.1524" layer="91"/>
-<pinref part="P7" gate="G$1" pin="1"/>
+<pinref part="M6" gate="G$1" pin="1"/>
 </segment>
 </net>
@@
 <pinref part="U10" gate="G$1" pin="OUT-"/>
 <wire x1="226.06" y1="25.4" x2="236.22" y2="25.4" width="0.1524" layer="91"/>
-<pinref part="P7" gate="G$1" pin="2"/>
+<pinref part="M6" gate="G$1" pin="2"/>
 </segment>
 </net>
@@
 <pinref part="U11" gate="G$1" pin="OUT+"/>
 <wire x1="226.06" y1="-15.24" x2="236.22" y2="-15.24" width="0.1524" layer="91"/>
-<pinref part="P6" gate="G$1" pin="1"/>
+<pinref part="M7" gate="G$1" pin="1"/>
 </segment>
 </net>
@@
 <pinref part="U11" gate="G$1" pin="OUT-"/>
 <wire x1="226.06" y1="-17.78" x2="236.22" y2="-17.78" width="0.1524" layer="91"/>
-<pinref part="P6" gate="G$1" pin="2"/>
+<pinref part="M7" gate="G$1" pin="2"/>
 </segment>
 </net>
@@
 <pinref part="U4" gate="G$1" pin="OUT-"/>
 <wire x1="140.462" y1="91.44" x2="139.7" y2="91.44" width="0.1524" layer="91"/>
-<pinref part="P2" gate="G$1" pin="2"/>
+<pinref part="M0" gate="G$1" pin="2"/>
 <wire x1="139.7" y1="91.44" x2="132.08" y2="91.44" width="0.1524" layer="91"/>
 <junction x="139.7" y="91.44"/>

Commit message: Board RC1
Parts:
- MI: value B2B-PH-K -> B2B-PH-K-S(LF)(SN)
- U12: value TCA9548APWR -> TCA9548APWR | PCA9548APW,118 | PI4MSD5V9547LEX
Other:
- note added: "3.3kohm resistor ladder"
Changed lines of the file:
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@@
 <part name="U$63" library="microbuilder" deviceset="GND" device=""/>
 <part name="U$65" library="microbuilder" deviceset="FRAME_A4_ADAFRUIT" device=""/>
-<part name="U12" library="microbuilder" deviceset="TCA9548A" device="" value=" TCA9548APWR"/>
+<part name="U12" library="microbuilder" deviceset="TCA9548A" device="" value=" TCA9548APWR | PCA9548APW,118 | PI4MSD5V9547LEX"/>
 <part name="R5" library="microbuilder" deviceset="RESISTOR" device="0805_NOOUTLINE" value="10K"/>
 <part name="R6" library="microbuilder" deviceset="RESISTOR" device="0805_NOOUTLINE" value="10K"/>
@@
 <part name="U$17" library="microbuilder" deviceset="GND" device=""/>
 <part name="U$18" library="microbuilder" deviceset="GND" device=""/>
-<part name="MI" library="con-jst-ph" deviceset="B2B-PH-K" device=""/>
+<part name="MI" library="con-jst-ph" deviceset="B2B-PH-K" device="" value="B2B-PH-K-S(LF)(SN)"/>
 <part name="M0" library="con-jst-ph" deviceset="B2B-PH-K" device=""/>
 <part name="M1" library="con-jst-ph" deviceset="B2B-PH-K" device=""/>
@@
 <instance part="MI" gate="G$1" x="144.78" y="139.7" smashed="yes">
 <attribute name="NAME" x="143.51" y="142.875" size="1.778" layer="95"/>
-<attribute name="VALUE" x="143.51" y="132.08" size="1.778" layer="95"/>
+<attribute name="VALUE" x="150.368" y="139.7" size="1.778" layer="95"/>
 </instance>
 <instance part="M0" gate="G$1" x="144.78" y="93.98" smashed="yes">
@@
 <sheet>
 <plain>
+<text x="102.87" y="104.394" size="1.778" layer="97">3.3kohm resistor ladder</text>
 </plain>
 <instances>

Commit message: More improvements
Parts:
- removed CN1: 1X4-BIG, adafruit:1X4-BIG
- removed JP2: (no value), microbuilder:HEADER-1X576MIL_FULL
- added P1: B5B-PH-K, con-jst-ph:B5B-PH-K
- added P2: B4B-PH-K, con-jst-ph:B4B-PH-K
Connections:
- net +5V: now also P1.2, P2.1; no longer CN1.1, JP2.2
- net GND: now also P1.3, P2.2; no longer CN1.2, JP2.3
- net INPUTSCL: now also P1.5, P2.4; no longer CN1.4, JP2.5
- net INPUTSDA: now also P1.4, P2.3; no longer CN1.3, JP2.4
- net VIN: now also P1.1; no longer JP2.1
Other:
- note added: "NOTE: VIN is 3.3v"
Changed lines of the file:
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@@
 <class number="1" name="Ground" width="0.2032" drill="0.3048">
 </class>
-<class number="2" name="Power" width="0.2032" drill="0.3048">
+<class number="2" name="Power" width="0.3048" drill="0.3048">
 </class>
 </classes>
@@
 <part name="C6" library="microbuilder" deviceset="CAP_CERAMIC" device="0805-NOOUTLINE" value="1uF"/>
 <part name="U$22" library="microbuilder" deviceset="GND" device=""/>
-<part name="JP2" library="microbuilder" deviceset="HEADER-1X5" device="76MIL_FULL"/>
-<part name="U$23" library="microbuilder" deviceset="VIN" device=""/>
-<part name="U$24" library="microbuilder" deviceset="GND" device=""/>
 <part name="U4" library="microbuilder" deviceset="DRV2605" device="_SOP" value="DRV2605LDGS"/>
 <part name="U$26" library="microbuilder" deviceset="GND" device=""/>
@@
 <part name="P+8" library="supply1" library_urn="urn:adsk.eagle:library:371" deviceset="+5V" device=""/>
 <part name="P+9" library="supply1" library_urn="urn:adsk.eagle:library:371" deviceset="+5V" device=""/>
-<part name="P+10" library="supply1" library_urn="urn:adsk.eagle:library:371" deviceset="+5V" device=""/>
 <part name="P+11" library="supply1" library_urn="urn:adsk.eagle:library:371" deviceset="+5V" device=""/>
 <part name="U$8" library="microbuilder" deviceset="GND" device=""/>
-<part name="CN1" library="adafruit" library_urn="urn:adsk.eagle:library:420" deviceset="1X4" device="-BIG"/>
 <part name="U$10" library="microbuilder" deviceset="GND" device=""/>
 <part name="U$11" library="microbuilder" deviceset="GND" device=""/>
@@
 <part name="P+19" library="supply1" library_urn="urn:adsk.eagle:library:371" deviceset="+5V" device=""/>
 <part name="P+20" library="supply1" library_urn="urn:adsk.eagle:library:371" deviceset="+5V" device=""/>
+<part name="P1" library="con-jst-ph" deviceset="B5B-PH-K" device=""/>
+<part name="U$20" library="microbuilder" deviceset="VIN" device=""/>
+<part name="P+21" library="supply1" library_urn="urn:adsk.eagle:library:371" deviceset="+5V" device=""/>
+<part name="U$25" library="microbuilder" deviceset="GND" device=""/>
+<part name="P2" library="con-jst-ph" deviceset="B4B-PH-K" device=""/>
 </parts>
 <sheets>
@@
 <attribute name="VALUE" x="155.956" y="114.3" size="1.27" layer="96"/>
 </instance>
-<instance part="JP2" gate="A" x="40.64" y="88.9" smashed="yes">
-<attribute name="NAME" x="34.29" y="97.155" size="1.778" layer="95"/>
-<attribute name="VALUE" x="34.29" y="78.74" size="1.778" layer="96"/>
-</instance>
-<instance part="U$23" gate="G$1" x="30.48" y="101.6" smashed="yes">
-<attribute name="VALUE" x="28.956" y="102.616" size="1.27" layer="96"/>
-</instance>
-<instance part="U$24" gate="G$1" x="45.72" y="86.36" smashed="yes">
-<attribute name="VALUE" x="44.196" y="83.82" size="1.27" layer="96"/>
-</instance>
 <instance part="U4" gate="G$1" x="119.38" y="91.44" smashed="yes">
 <attribute name="NAME" x="109.22" y="109.22" size="1.27" layer="95"/>
@@
 <attribute name="VALUE" x="248.92" y="105.41" size="1.778" layer="96" rot="R90"/>
 </instance>
-<instance part="P+10" gate="1" x="25.4" y="101.6" smashed="yes">
-<attribute name="VALUE" x="22.86" y="96.52" size="1.778" layer="96" rot="R90"/>
-</instance>
 <instance part="P+11" gate="1" x="20.32" y="64.77" smashed="yes">
 <attribute name="VALUE" x="17.78" y="59.69" size="1.778" layer="96" rot="R90"/>
@@
 <instance part="U$8" gate="G$1" x="20.32" y="54.61" smashed="yes">
 <attribute name="VALUE" x="18.796" y="52.07" size="1.27" layer="96"/>
-</instance>
-<instance part="CN1" gate="G$1" x="35.56" y="58.42" smashed="yes">
-<attribute name="NAME" x="40.64" y="66.04" size="1.27" layer="95" font="vector" rot="R180"/>
-<attribute name="VALUE" x="35.56" y="48.26" size="1.27" layer="96" font="vector"/>
 </instance>
 <instance part="U$10" gate="G$1" x="104.14" y="127" smashed="yes">
@@
 <instance part="P+20" gate="1" x="198.12" y="128.27" smashed="yes">
 <attribute name="VALUE" x="195.58" y="123.19" size="1.778" layer="96" rot="R90"/>
+</instance>
+<instance part="P1" gate="G$1" x="41.148" y="115.824" smashed="yes">
+<attribute name="NAME" x="39.878" y="124.079" size="1.778" layer="95"/>
+<attribute name="VALUE" x="39.878" y="105.664" size="1.778" layer="95"/>
+</instance>
+<instance part="U$20" gate="G$1" x="26.67" y="128.524" smashed="yes">
+<attribute name="VALUE" x="25.146" y="129.54" size="1.27" layer="96"/>
+</instance>
+<instance part="P+21" gate="1" x="21.59" y="128.524" smashed="yes">
+<attribute name="VALUE" x="19.05" y="123.444" size="1.778" layer="96" rot="R90"/>
+</instance>
+<instance part="U$25" gate="G$1" x="47.498" y="113.284" smashed="yes">
+<attribute name="VALUE" x="45.974" y="110.744" size="1.27" layer="96"/>
+</instance>
+<instance part="P2" gate="G$1" x="36.322" y="55.88" smashed="yes">
+<attribute name="NAME" x="35.052" y="64.135" size="1.778" layer="95"/>
+<attribute name="VALUE" x="35.052" y="48.26" size="1.778" layer="95"/>
 </instance>
 </instances>
@@
 </segment>
 </net>
-<net name="VIN" class="2">
-<segment>
-<pinref part="JP2" gate="A" pin="1"/>
-<pinref part="U$23" gate="G$1" pin="VIN"/>
-<wire x1="38.1" y1="93.98" x2="30.48" y2="93.98" width="0.1524" layer="91"/>
-<wire x1="30.48" y1="93.98" x2="30.48" y2="99.06" width="0.1524" layer="91"/>
+<net name="VIN" class="0">
+<segment>
+<pinref part="U$20" gate="G$1" pin="VIN"/>
+<wire x1="36.068" y1="120.904" x2="26.67" y2="120.904" width="0.1524" layer="91"/>
+<wire x1="26.67" y1="120.904" x2="26.67" y2="125.984" width="0.1524" layer="91"/>
+<pinref part="P1" gate="G$1" pin="1"/>
 </segment>
 </net>
@@
 </segment>
 <segment>
-<pinref part="U$24" gate="G$1" pin="GND"/>
-<pinref part="JP2" gate="A" pin="3"/>
-<wire x1="45.72" y1="88.9" x2="38.1" y2="88.9" width="0.1524" layer="91"/>
-</segment>
-<segment>
 <pinref part="U$8" gate="G$1" pin="GND"/>
 <wire x1="20.32" y1="57.15" x2="20.32" y2="58.42" width="0.1524" layer="91"/>
-<wire x1="20.32" y1="58.42" x2="30.48" y2="58.42" width="0.1524" layer="91"/>
-<pinref part="CN1" gate="G$1" pin="2"/>
+<wire x1="20.32" y1="58.42" x2="31.242" y2="58.42" width="0.1524" layer="91"/>
+<pinref part="P2" gate="G$1" pin="2"/>
 </segment>
 <segment>
@@
 <pinref part="U$18" gate="G$1" pin="GND"/>
 <pinref part="U8" gate="G$1" pin="IN/TRIG"/>
+</segment>
+<segment>
+<pinref part="P1" gate="G$1" pin="3"/>
+<pinref part="U$25" gate="G$1" pin="GND"/>
+<wire x1="36.068" y1="115.824" x2="47.498" y2="115.824" width="0.1524" layer="91"/>
 </segment>
 </net>
@@
 <net name="INPUTSDA" class="0">
 <segment>
-<pinref part="JP2" gate="A" pin="4"/>
-<wire x1="38.1" y1="86.36" x2="25.4" y2="86.36" width="0.1524" layer="91"/>
-<label x="21.59" y="86.36" size="1.778" layer="95"/>
-</segment>
-<segment>
-<wire x1="30.48" y1="55.88" x2="24.13" y2="55.88" width="0.1524" layer="91"/>
-<pinref part="CN1" gate="G$1" pin="3"/>
+<wire x1="31.242" y1="55.88" x2="24.13" y2="55.88" width="0.1524" layer="91"/>
 <label x="22.86" y="55.88" size="1.778" layer="95"/>
+<pinref part="P2" gate="G$1" pin="3"/>
 </segment>
 <segment>
@@
 <label x="97.79" y="139.7" size="1.778" layer="95"/>
 </segment>
+<segment>
+<wire x1="36.068" y1="113.284" x2="21.59" y2="113.284" width="0.1524" layer="91"/>
+<label x="17.78" y="113.284" size="1.778" layer="95"/>
+<pinref part="P1" gate="G$1" pin="4"/>
+</segment>
 </net>
 <net name="INPUTSCL" class="0">
 <segment>
-<pinref part="JP2" gate="A" pin="5"/>
-<wire x1="38.1" y1="83.82" x2="25.4" y2="83.82" width="0.1524" layer="91"/>
-<label x="21.59" y="83.82" size="1.778" layer="95"/>
-</segment>
-<segment>
-<wire x1="30.48" y1="53.34" x2="24.13" y2="53.34" width="0.1524" layer="91"/>
-<pinref part="CN1" gate="G$1" pin="4"/>
+<wire x1="31.242" y1="53.34" x2="24.13" y2="53.34" width="0.1524" layer="91"/>
 <label x="22.86" y="53.34" size="1.778" layer="95"/>
+<pinref part="P2" gate="G$1" pin="4"/>
 </segment>
 <segment>
@@
 <wire x1="106.68" y1="137.16" x2="92.71" y2="137.16" width="0.1524" layer="91"/>
 <label x="97.79" y="137.16" size="1.778" layer="95"/>
+</segment>
+<segment>
+<wire x1="36.068" y1="110.744" x2="21.59" y2="110.744" width="0.1524" layer="91"/>
+<label x="17.78" y="110.744" size="1.778" layer="95"/>
+<pinref part="P1" gate="G$1" pin="5"/>
 </segment>
 </net>
@@
 </segment>
 <segment>
-<pinref part="P+10" gate="1" pin="+5V"/>
-<wire x1="25.4" y1="99.06" x2="25.4" y2="91.44" width="0.1524" layer="91"/>
-<pinref part="JP2" gate="A" pin="2"/>
-<wire x1="25.4" y1="91.44" x2="38.1" y2="91.44" width="0.1524" layer="91"/>
-</segment>
-<segment>
 <pinref part="P+11" gate="1" pin="+5V"/>
 <wire x1="20.32" y1="62.23" x2="20.32" y2="60.96" width="0.1524" layer="91"/>
-<wire x1="20.32" y1="60.96" x2="30.48" y2="60.96" width="0.1524" layer="91"/>
-<pinref part="CN1" gate="G$1" pin="1"/>
+<wire x1="20.32" y1="60.96" x2="31.242" y2="60.96" width="0.1524" layer="91"/>
+<pinref part="P2" gate="G$1" pin="1"/>
 </segment>
 <segment>
@@
 <junction x="198.12" y="125.73"/>
 </segment>
+<segment>
+<pinref part="P+21" gate="1" pin="+5V"/>
+<wire x1="21.59" y1="125.984" x2="21.59" y2="118.364" width="0.1524" layer="91"/>
+<wire x1="21.59" y1="118.364" x2="36.068" y2="118.364" width="0.1524" layer="91"/>
+<pinref part="P1" gate="G$1" pin="2"/>
+</segment>
 </net>
 </nets>
@@
 <plain>
 <text x="102.87" y="104.394" size="1.778" layer="97">3.3kohm resistor ladder</text>
+<text x="55.626" y="118.618" size="3.81" layer="97">NOTE: VIN is 3.3v</text>
 </plain>
 <instances>
@@
 </segment>
 </net>
-<net name="VIN" class="2">
+<net name="VIN" class="0">
 <segment>
 <pinref part="R6" gate="G$1" pin="2"/>
